File: PCBs/Melodica_main/V2/melodica_main.kicad_pcb (KiCad board)
At the start: 2 copper layers, 197 x 40 mm, 38 parts, among them J1 AudioJack3_SwitchTR, U1 STM32F405RGTx

Commit message: V2 PCB design of melodica
Parts:
- moved C7 92.9 mm to (71.0, 103.5)
- moved C5 91.6 mm to (55.5, 104.0)
- moved 1k3 87.0 mm to (55.0, 116.3), turned to 90 degrees
- moved 1k4 87.0 mm to (55.0, 119.5), turned to -90 degrees
- moved Reset2 86.5 mm to (59.0, 122.8)
- moved U1 76.0 mm to (64.5, 112.0)
- moved Programmer2 74.4 mm to (67.5, 101.5), turned to -90 degrees
- moved C6 73.0 mm to (71.0, 121.5)
- moved Leave_Open2 72.8 mm to (68.5, 128.5)
- moved J1 61.2 mm to (44.0, 116.0), turned to -90 degrees
- moved 3.6k 7.31 mm to (198.2, 106.5)
- moved 3.6k 6.66 mm to (205.8, 109.0)
- moved 3.6k 6.01 mm to (198.2, 111.5)
- moved BT1 4.47 mm to (211.5, 108.9)
- renumbered 220R2 to 220, 220R1 to 220R, 3.6k1 to 3.6k, 3.6k2 to 3.6k, 3.6k3 to 3.6k, Leave_Open1 to Open
Routing:
- net /UART_RX_MAIN: track 40.8 -> 273.8 mm
- net /UART_RX_SYNTH: track 83.0 -> 239.9 mm
- net GND: track 511.3 -> 561.6 mm, vias 14 -> 20
- net VCC: track 383.5 -> 429.1 mm
- net Net-(U1-BOOT0): track 0.00 -> 34.8 mm, vias 0 -> 1
- net Net-(U1-NRST): track 0.00 -> 30.9 mm
- net /DAC2_SYNTH: track 0.00 -> 20.5 mm, vias 0 -> 1
- net /DAC1_SYNTH: track 0.00 -> 16.4 mm, vias 0 -> 1
- net /SWDIO_SYNTH: track 0.00 -> 10.5 mm, vias 0 -> 1
- net Net-(U1-VCAP_2): track 0.00 -> 7.32 mm, vias 0 -> 1
- net Net-(U1-VCAP_1): track 0.00 -> 5.76 mm
- net /SWCLK_SYNTH: track 0.00 -> 5.12 mm
- net Net-(BT1-+): track 42.4 -> 37.6 mm
- net /IN_1: track 172.3 -> 169.5 mm
- net /IN_2: track 123.2 -> 125.2 mm
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Other:
- board size 197 x 40 mm -> 178.5 x 32.5 mm
- board text added: "Electric Melodica V2.0"
- board text removed: "Electric Melodica V1.0"
