File: PCBs/Melodica_main/V2/melodica_main.kicad_sch (KiCad schematic)
At the start: 38 parts, among them J1 AudioJack3_SwitchTR, U1 STM32F405RGTx

Commit message: V2 PCB design of melodica
Other:
- note added: "<- NOTE: SWCLK and SWDIO pins are flipped accidentally here, leaving as is but in future pcb prints this should be fixed"
Changed lines of the file:
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@@
+		)
+	)
+	(text "<- NOTE: SWCLK and SWDIO pins are flipped accidentally here, leaving as is but in future pcb prints this should be fixed"
+		(exclude_from_sim no)
+		(at 295.91 108.712 0)
+		(effects
+			(font
+				(size 1.27 1.27)
+			)
 		)
 	)
